File: PCB-Layouts/MoleNet_v2/MoleNet_v2.brd (EAGLE design)
At the start: 76.5 x 67.6 mm, 31 parts, among them IC1 25LC080P, Q1 BS250, Q2 BS170, U1 MCP1703-5002E/DB, U2 ATMEGA328P-PU, U3 RFM69CW, X1 SMA-142-0711-821/826

Commit message: added/corrected part values in all layouts; created partlist for version 2.1
Parts:
- C1: value 10uF -> 4.7uF
- C10, C11, C12, C4, C5, C6, C9: value (none) -> 100nF
- C2, C3: value (none) -> 1uF
- C7, C8: value (none) -> 22pF
- Q3: value (none) -> 8MHz
- R1: value (none) -> 10k
- R2: value (none) -> 100k
Changed lines of the file:
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@@
 <attribute name="NAME" x="6.985" y="32.7025" size="1.27" layer="25" ratio="10"/>
 </element>
-<element name="R2" library="resistor" package="0207/10" value="" x="2.8575" y="43.18" smashed="yes" rot="R90">
+<element name="R2" library="resistor" package="0207/10" value="100k" x="2.8575" y="43.18" smashed="yes" rot="R90">
 <attribute name="NAME" x="4.572" y="43.1165" size="1.27" layer="25" ratio="10"/>
 <attribute name="VALUE" x="3.4925" y="40.9194" size="1.27" layer="27" ratio="10" rot="R90"/>
@@
 <attribute name="VALUE" x="49.3256" y="30.305" size="1.27" layer="27" rot="R180"/>
 </element>
-<element name="C1" library="resistor" package="E2,5-6" value="10uF" x="4.1275" y="52.07" smashed="yes" rot="R180">
+<element name="C1" library="resistor" package="E2,5-6" value="4.7uF" x="4.1275" y="52.07" smashed="yes" rot="R180">
 <attribute name="NAME" x="1.0795" y="54.864" size="1.27" layer="25" ratio="10"/>
 <attribute name="VALUE" x="1.4605" y="54.737" size="1.27" layer="27" ratio="10" rot="R180"/>
 </element>
-<element name="C2" library="resistor" package="C025-025X050" value="" x="9.2075" y="48.26" smashed="yes" rot="R90">
+<element name="C2" library="resistor" package="C025-025X050" value="1uF" x="9.2075" y="48.26" smashed="yes" rot="R90">
 <attribute name="NAME" x="7.874" y="44.3865" size="1.27" layer="25" ratio="10"/>
 <attribute name="VALUE" x="12.0015" y="45.974" size="1.27" layer="27" ratio="10" rot="R90"/>
 </element>
-<element name="C3" library="resistor" package="C025-025X050" value="" x="21.6027" y="48.26" smashed="yes" rot="R90">
+<element name="C3" library="resistor" package="C025-025X050" value="1uF" x="21.6027" y="48.26" smashed="yes" rot="R90">
 <attribute name="NAME" x="21.844" y="51.0413" size="1.27" layer="25" ratio="10"/>
 <attribute name="VALUE" x="24.3967" y="45.974" size="1.27" layer="27" ratio="10" rot="R90"/>
 </element>
-<element name="C4" library="resistor" package="C025-025X050" value="" x="40.9575" y="35.56" smashed="yes">
+<element name="C4" library="resistor" package="C025-025X050" value="100nF" x="40.9575" y="35.56" smashed="yes">
 <attribute name="NAME" x="43.7515" y="34.544" size="1.27" layer="25" ratio="10"/>
 <attribute name="VALUE" x="38.6715" y="32.766" size="1.27" layer="27" ratio="10"/>
 </element>
-<element name="C6" library="resistor" package="C025-025X050" value="" x="40.9575" y="38.100003125" smashed="yes">
+<element name="C6" library="resistor" package="C025-025X050" value="100nF" x="40.9575" y="38.100003125" smashed="yes">
 <attribute name="NAME" x="43.7515" y="38.354003125" size="1.27" layer="25" ratio="10"/>
 <attribute name="VALUE" x="38.6715" y="35.306003125" size="1.27" layer="27" ratio="10"/>
@@
 <attribute name="VALUE" x="72.5043" y="16.3322" size="1.778" layer="27" rot="R180"/>
 </element>
-<element name="C5" library="resistor" package="C025-025X050" value="" x="25.5016" y="40.6527" smashed="yes" rot="R180">
+<element name="C5" library="resistor" package="C025-025X050" value="100nF" x="25.5016" y="40.6527" smashed="yes" rot="R180">
 <attribute name="NAME" x="23.0251" y="39.3192" size="1.27" layer="25" ratio="10" rot="R90"/>
 <attribute name="VALUE" x="27.7876" y="43.4467" size="1.27" layer="27" ratio="10" rot="R180"/>
@@
 <attribute name="VALUE" x="24.4475" y="64.135" size="1.27" layer="27" rot="R180"/>
 </element>
-<element name="C10" library="resistor" package="C025-025X050" value="" x="23.1775" y="57.15" smashed="yes" rot="R90">
+<element name="C10" library="resistor" package="C025-025X050" value="100nF" x="23.1775" y="57.15" smashed="yes" rot="R90">
 <attribute name="NAME" x="25.654" y="58.3565" size="1.27" layer="25" ratio="10"/>
 <attribute name="VALUE" x="25.9715" y="54.864" size="1.27" layer="27" ratio="10" rot="R90"/>
 </element>
-<element name="R1" library="resistor" package="0207/10" value="" x="15.5575" y="55.88" smashed="yes" rot="R180">
+<element name="R1" library="resistor" package="0207/10" value="10k" x="15.5575" y="55.88" smashed="yes" rot="R180">
 <attribute name="NAME" x="11.8745" y="57.404" size="1.27" layer="25" ratio="10"/>
 <attribute name="VALUE" x="17.8181" y="56.515" size="1.27" layer="27" ratio="10" rot="R180"/>
 </element>
-<element name="Q3" library="crystal" package="HC18U-V" value="" x="24.4475" y="33.02" smashed="yes" rot="R270">
+<element name="Q3" library="crystal" package="HC18U-V" value="8MHz" x="24.4475" y="33.02" smashed="yes" rot="R270">
 <attribute name="OC_FARNELL" value="unknown" x="24.4475" y="33.02" size="1.778" layer="27" rot="R270" display="off"/>
 <attribute name="MF" value="" x="24.4475" y="33.02" size="1.778" layer="27" rot="R270" display="off"/>
@@
 <attribute name="VALUE" x="19.8247" y="38.1" size="1.27" layer="27" ratio="10" rot="R270"/>
 </element>
-<element name="C7" library="resistor" package="C025-025X050" value="" x="18.0975" y="35.56" smashed="yes" rot="R180">
+<element name="C7" library="resistor" package="C025-025X050" value="22pF" x="18.0975" y="35.56" smashed="yes" rot="R180">
 <attribute name="NAME" x="12.6365" y="34.544" size="1.27" layer="25" ratio="10"/>
 <attribute name="VALUE" x="20.3835" y="38.354" size="1.27" layer="27" ratio="10" rot="R180"/>
 </element>
-<element name="C8" library="resistor" package="C025-025X050" value="" x="18.0975" y="30.48" smashed="yes" rot="R180">
+<element name="C8" library="resistor" package="C025-025X050" value="22pF" x="18.0975" y="30.48" smashed="yes" rot="R180">
 <attribute name="NAME" x="12.6365" y="29.464" size="1.27" layer="25" ratio="10"/>
 <attribute name="VALUE" x="20.3835" y="33.274" size="1.27" layer="27" ratio="10" rot="R180"/>
@@
 <attribute name="VALUE" x="50.4825" y="39.37" size="1.27" layer="27" rot="R90"/>
 </element>
-<element name="C9" library="resistor" package="C025-025X050" value="" x="30.48" y="12.7" smashed="yes" rot="R270">
+<element name="C9" library="resistor" package="C025-025X050" value="100nF" x="30.48" y="12.7" smashed="yes" rot="R270">
 <attribute name="NAME" x="29.464" y="9.906" size="1.27" layer="25" ratio="10" rot="R270"/>
 <attribute name="VALUE" x="27.686" y="14.986" size="1.27" layer="27" ratio="10" rot="R270"/>
 </element>
-<element name="C11" library="resistor" package="C025-025X050" value="" x="20.32" y="2.54"/>
-<element name="C12" library="resistor" package="C025-025X050" value="" x="8.89" y="24.13" rot="R90"/>
+<element name="C11" library="resistor" package="C025-025X050" value="100nF" x="20.32" y="2.54"/>
+<element name="C12" library="resistor" package="C025-025X050" value="100nF" x="8.89" y="24.13" rot="R90"/>
 <element name="JP2" library="pinhead" package="2X03" value="" x="38.1" y="16.51" rot="R180"/>
 <element name="JP5" library="pinhead" package="1X04" value="" x="40.005" y="46.99" rot="R270"/>
