File: PCB-Layouts/MoleNet_v21/MoleNet_v21.brd (EAGLE design)
At the start: 76.5 x 67.6 mm, 31 parts, among them IC1 25LC080P, Q1 BS250, Q2 BS170, U1 MCP1703-5002E/DB, U2 ATMEGA328P-PU, U3 RFM69CW, X1 SMA-142-0711-821/826

Commit message: MoleNet version 2.1 ready
Parts:
- added JP7: (no value), pinhead:1X06
- added JP8: (no value), pinhead:1X03
- JP3: value ISP -> (none); device pinhead:2X05 -> pinhead:1X03
- JP4: device pinhead:1X04 -> pinhead:1X03
- JP6: value (none) -> ISP; device pinhead:1X06 -> pinhead:2X05
- moved JP3 39.9 mm to (6.35, 41.9), turned to 270 degrees
- moved JP6 32.9 mm to (46.0, 45.7), turned to 90 degrees
- moved C9 14.5 mm to (44.5, 8.89)
- moved IC1 14.5 mm to (38.1, 6.35)
- moved Q1 10.2 mm to (5.40, 25.4)
- moved Q2 10.2 mm to (9.21, 30.5)
- moved R2 10.2 mm to (2.86, 33.0)
- moved JP4 5.40 mm to (24.1, 17.8), turned to 90 degrees
- moved C11 5.24 mm to (19.1, 7.62), turned to 90 degrees
- moved C12 2.84 mm to (10.2, 21.6), turned to 180 degrees
- moved X1 0.25 mm to (74.0, 7.44)
- moved JP5 0.13 mm to (40.1, 47.0)
Connections:
- new net N$2: JP3.2, Q1.S, R2.2
- new net SENSRXD: C11.1, JP8.3, K1.3
- net +12V: now also JP3.1; no longer Q1.S, R2.2
- net D4: now also JP4.3; no longer JP4.4
- net D5: now also JP4.2; no longer JP4.3
- net D6: now also JP4.1; no longer JP4.2
- net D8: now also JP8.1; no longer JP4.1
- net GND: now also JP6.10, JP6.4, JP6.8, JP7.5, JP7.6; no longer JP3.10, JP3.4, JP3.6, JP3.8, JP6.5
- net MISO: now also JP6.9; no longer JP3.9
- net MOSI: now also JP6.1; no longer JP3.1
- net N$9: now also JP7.1; no longer JP6.1
- net RESET: now also JP6.5; no longer JP3.5
- net RXD: now also JP7.3, JP8.2; no longer C11.1, JP6.3, K1.3
- net SCK: now also JP6.7; no longer JP3.7
- net TXD: now also JP7.2; no longer JP6.2
- net VCC: now also JP3.3, JP6.2, JP7.4; no longer JP3.2, JP6.4
Routing:
- net MISOSW: track 54.0 -> 28.1 mm
- net N$2: track 0.00 -> 19.2 mm
- net VCC: track 276.9 -> 258.2 mm, vias 2 -> 3
- net SCKSW: track 63.7 -> 49.1 mm
- net N$10: track 25.1 -> 13.5 mm
- net SENSRXD: track 0.00 -> 11.5 mm
- net D8: track 4.26 -> 15.2 mm
- net +12V: track 35.9 -> 25.7 mm
- net D7: track 30.5 -> 21.1 mm
- net RXD: track 78.2 -> 70.0 mm
- net D9: track 23.3 -> 16.6 mm, vias 1 -> 0
- net D6: track 10.2 -> 16.2 mm, vias 0 -> 1
- net D5: track 14.9 -> 20.5 mm
- net MOSISW: track 57.9 -> 53.2 mm
- net NSS: track 39.1 -> 34.8 mm
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
Commit message: MoleNet version 2.1 rtm
Parts:
- moved JP8 26.7 mm to (12.7, 33.0), turned to 90 degrees
- moved JP2 14.4 mm to (27.9, 6.35), turned to 270 degrees
- moved Q2 5.24 mm to (10.5, 25.4)
- moved JP4 4.58 mm to (20.3, 15.2), turned to 270 degrees
- moved C1 4.02 mm to (5.40, 48.3)
- moved C12 3.59 mm to (12.7, 19.1), turned to 0 degrees
- moved JP5 3.10 mm to (41.9, 44.5)
- moved R2 2.84 mm to (4.13, 30.5)
- moved Q3 2.84 mm to (25.7, 30.5)
- moved C10 2.84 mm to (24.4, 54.6)
- moved JP3 2.84 mm to (7.62, 39.4)
- moved Q1 2.84 mm to (6.67, 22.9)
- moved R1 2.84 mm to (16.8, 53.3)
- moved U1 2.84 mm to (16.3, 46.2)
- moved C2 2.84 mm to (10.5, 45.7)
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Connections:
- net RXD: now also JP8.3; no longer JP8.2
- net SENSRXD: now also JP8.2; no longer JP8.3
Routing:
- net VCC: track 258.2 -> 217.7 mm, vias 3 -> 2
- net RXD: track 70.0 -> 36.6 mm
- net D2: track 79.2 -> 47.7 mm
- net SENSRXD: track 11.5 -> 41.7 mm
- net MISO: track 50.5 -> 79.6 mm
- net SCK: track 45.7 -> 68.8 mm
- net NSS: track 34.8 -> 54.0 mm, vias 0 -> 1
- net SCKSW: track 49.1 -> 63.4 mm, vias 0 -> 2
- net MOSI: track 37.3 -> 50.6 mm
- net D8: track 15.2 -> 25.7 mm, vias 0 -> 1
- net MOSISW: track 53.2 -> 62.6 mm, vias 1 -> 2
- net D4: track 31.2 -> 39.5 mm
- net TXD: track 26.8 -> 20.3 mm, vias 0 -> 1
- net D3: track 55.0 -> 51.0 mm
- net D5: track 20.5 -> 24.2 mm
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Other:
- board size 76.5 x 67.6 mm -> 74 x 63.8 mm

Commit message: v2.1 now really rtm :-)
Routing:
- net VCC: track 217.7 -> 207.1 mm
Changed lines of the file:
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@@
 <setting verticaltext="up"/>
 </settings>
-<grid distance="25" unitdist="mil" unit="mil" style="lines" multiple="1" display="yes" altdistance="0.025" altunitdist="inch" altunit="inch"/>
+<grid distance="50" unitdist="mil" unit="mil" style="lines" multiple="1" display="yes" altdistance="0.025" altunitdist="inch" altunit="inch"/>
 <layers>
 <layer number="1" name="Top" color="4" fill="1" visible="yes" active="yes"/>
@@
 <via x="63.8175" y="7.62" extent="1-16" drill="0.5" shape="square"/>
 <via x="63.8175" y="4.064" extent="1-16" drill="0.5" shape="square"/>
-<via x="49.0855" y="13.462" extent="1-16" drill="0.5" shape="square"/>
-<via x="49.0855" y="10.922" extent="1-16" drill="0.5" shape="square"/>
+<via x="49.0855" y="14.732" extent="1-16" drill="0.5" shape="square"/>
+<via x="49.0855" y="12.192" extent="1-16" drill="0.5" shape="square"/>
 <via x="49.0855" y="8.382" extent="1-16" drill="0.5" shape="square"/>
 <via x="59.69" y="14.7955" extent="1-16" drill="0.5" shape="square"/>
@@
 <wire x1="16.8275" y1="58.42" x2="16.8275" y2="54.9275" width="0.6096" layer="1"/>
 <wire x1="46.99" y1="35.56" x2="53.34" y2="35.56" width="0.6096" layer="1"/>
-<wire x1="53.34" y1="35.56" x2="56.515" y2="35.56" width="0.6096" layer="1"/>
-<wire x1="56.515" y1="35.56" x2="60.0075" y2="39.0525" width="0.6096" layer="1"/>
 <wire x1="22.8727" y1="44.45" x2="22.225" y2="44.45" width="0.6096" layer="1"/>
 <wire x1="22.225" y1="44.45" x2="20.32" y2="46.355" width="0.6096" layer="1"/>
@@
 <wire x1="10.795" y1="38.1" x2="9.525" y2="36.83" width="0.6096" layer="1"/>
 <wire x1="9.525" y1="36.83" x2="7.62" y2="36.83" width="0.6096" layer="1"/>
-<wire x1="60.0075" y1="54.2925" x2="53.34" y2="60.96" width="0.6096" layer="1"/>
-<wire x1="53.34" y1="60.96" x2="30.48" y2="60.96" width="0.6096" layer="1"/>
-<wire x1="30.48" y1="60.96" x2="27.94" y2="58.42" width="0.6096" layer="1"/>
-<wire x1="27.94" y1="58.42" x2="27.94" y2="45.72" width="0.6096" layer="1"/>
+<wire x1="60.0075" y1="54.2925" x2="55.88" y2="58.42" width="0.6096" layer="1"/>
+<wire x1="55.88" y1="58.42" x2="30.48" y2="58.42" width="0.6096" layer="1"/>
+<wire x1="30.48" y1="58.42" x2="27.94" y2="55.88" width="0.6096" layer="1"/>
+<wire x1="27.94" y1="55.88" x2="27.94" y2="45.72" width="0.6096" layer="1"/>
 <wire x1="27.94" y1="45.72" x2="26.67" y2="44.45" width="0.6096" layer="1"/>
 <wire x1="26.67" y1="44.45" x2="22.8727" y2="44.45" width="0.6096" layer="1"/>
-<wire x1="60.0075" y1="52.07" x2="60.0075" y2="39.0525" width="0.6096" layer="1"/>
 <wire x1="60.0075" y1="52.07" x2="60.0075" y2="54.2925" width="0.6096" layer="1"/>
 <wire x1="22.86" y1="38.1" x2="27.8511" y2="38.1" width="0.6096" layer="1"/>
@@
 <wire x1="46.99" y1="35.56" x2="45.72" y2="36.83" width="0.6096" layer="1"/>
 <wire x1="45.72" y1="36.83" x2="45.72" y2="38.1" width="0.6096" layer="1"/>
-<wire x1="44.45" y1="10.16" x2="45.72" y2="10.16" width="0.6096" layer="16"/>
-<wire x1="45.72" y1="10.16" x2="46.99" y2="11.43" width="0.6096" layer="16"/>
-<wire x1="46.99" y1="11.43" x2="46.99" y2="16.51" width="0.6096" layer="16"/>
-<wire x1="46.99" y1="16.51" x2="46.99" y2="23.1794" width="0.6096" layer="16"/>
+<wire x1="44.45" y1="10.16" x2="46.99" y2="10.16" width="0.6096" layer="16"/>
+<wire x1="46.99" y1="10.16" x2="46.99" y2="23.1794" width="0.6096" layer="16"/>
 <wire x1="46.99" y1="23.1794" x2="48.5756" y2="24.765" width="0.6096" layer="16"/>
-<wire x1="60.96" y1="10.16" x2="60.96" y2="15.875" width="0.6096" layer="16"/>
-<wire x1="60.96" y1="15.875" x2="60.325" y2="16.51" width="0.6096" layer="16"/>
-<wire x1="60.325" y1="16.51" x2="46.99" y2="16.51" width="0.6096" layer="16"/>
+<wire x1="60.0075" y1="52.07" x2="60.0075" y2="42.2275" width="0.6096" layer="1"/>
+<wire x1="60.0075" y1="42.2275" x2="53.34" y2="35.56" width="0.6096" layer="1"/>
+<wire x1="60.96" y1="10.16" x2="46.99" y2="10.16" width="0.6096" layer="16"/>
 </signal>
 <signal name="MISOSW">
@@
 <contactref element="IC1" pad="5"/>
 <wire x1="62.452" y1="15.462" x2="58.7375" y2="11.7475" width="0.6096" layer="1"/>
-<via x="58.7375" y="11.7475" extent="1-16" drill="0.6" shape="square"/>
 <contactref element="JP2" pad="2"/>
 <wire x1="62.452" y1="15.462" x2="66.9995" y2="15.462" width="0.6096" layer="1"/>
-<wire x1="58.7375" y1="11.7475" x2="58.7375" y2="4.1275" width="0.6096" layer="16"/>
+<wire x1="58.7375" y1="11.7475" x2="58.7375" y2="4.1275" width="0.6096" layer="1"/>
 <wire x1="58.7375" y1="4.1275" x2="57.15" y2="2.54" width="0.6096" layer="16"/>
 <wire x1="57.15" y1="2.54" x2="41.8973" y2="2.54" width="0.6096" layer="16"/>
@@
 <wire x1="36.83" y1="5.08" x2="39.37" y2="2.54" width="0.6096" layer="16"/>
 <wire x1="39.37" y1="2.54" x2="41.8973" y2="2.54" width="0.6096" layer="16"/>
+<via x="58.7375" y="4.1275" extent="1-16" drill="0.6" shape="square"/>
 </signal>
 <signal name="SCKSW">

Commit message: added/corrected part values in all layouts; created partlist for version 2.1
Parts:
- C1: value 10uF -> 4.7uF
- C10, C11, C12, C4, C5, C6, C9: value (none) -> 100nF
- C2, C3: value (none) -> 1uF
- C7, C8: value (none) -> 22pF
- L1: value (none) -> 10mH
- Q3: value (none) -> 8MHz
- R1: value (none) -> 10k
- R2: value (none) -> 100k
Changed lines of the file:
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@@
 <attribute name="NAME" x="4.445" y="18.7325" size="1.27" layer="25" ratio="10"/>
 </element>
-<element name="R2" library="resistor" package="0207/10" value="" x="4.1275" y="30.48" smashed="yes" rot="R90">
+<element name="R2" library="resistor" package="0207/10" value="100k" x="4.1275" y="30.48" smashed="yes" rot="R90">
 <attribute name="NAME" x="5.842" y="30.4165" size="1.27" layer="25" ratio="10"/>
 <attribute name="VALUE" x="4.7625" y="28.2194" size="1.27" layer="27" ratio="10" rot="R90"/>
@@
 <attribute name="VALUE" x="71.6915" y="55.118" size="1.27" layer="27" rot="R180"/>
 </element>
-<element name="L1" library="inductor-neosid" package="BS11" value="" x="46.0756" y="24.765" smashed="yes" rot="R180">
+<element name="L1" library="inductor-neosid" package="BS11" value="10mH" x="46.0756" y="24.765" smashed="yes" rot="R180">
 <attribute name="OC_FARNELL" value="unknown" x="46.0756" y="24.765" size="1.778" layer="27" rot="R180" display="off"/>
 <attribute name="MF" value="" x="46.0756" y="24.765" size="1.778" layer="27" rot="R180" display="off"/>
@@
 <attribute name="VALUE" x="49.3256" y="27.765" size="1.27" layer="27" rot="R180"/>
 </element>
-<element name="C1" library="resistor" package="E2,5-6" value="10uF" x="5.3975" y="48.26" smashed="yes" rot="R180">
+<element name="C1" library="resistor" package="E2,5-6" value="4.7uF" x="5.3975" y="48.26" smashed="yes" rot="R180">
 <attribute name="NAME" x="2.3495" y="51.054" size="1.27" layer="25" ratio="10"/>
 <attribute name="VALUE" x="2.7305" y="50.927" size="1.27" layer="27" ratio="10" rot="R180"/>
 </element>
-<element name="C2" library="resistor" package="C025-025X050" value="" x="10.4775" y="45.72" smashed="yes" rot="R90">
+<element name="C2" library="resistor" package="C025-025X050" value="1uF" x="10.4775" y="45.72" smashed="yes" rot="R90">
 <attribute name="NAME" x="9.144" y="41.8465" size="1.27" layer="25" ratio="10"/>
 <attribute name="VALUE" x="13.2715" y="43.434" size="1.27" layer="27" ratio="10" rot="R90"/>
 </element>
-<element name="C3" library="resistor" package="C025-025X050" value="" x="22.8727" y="45.72" smashed="yes" rot="R90">
+<element name="C3" library="resistor" package="C025-025X050" value="1uF" x="22.8727" y="45.72" smashed="yes" rot="R90">
 <attribute name="NAME" x="23.114" y="48.5013" size="1.27" layer="25" ratio="10"/>
 <attribute name="VALUE" x="25.6667" y="43.434" size="1.27" layer="27" ratio="10" rot="R90"/>
 </element>
-<element name="C4" library="resistor" package="C025-025X050" value="" x="41.9227" y="33.02" smashed="yes">
+<element name="C4" library="resistor" package="C025-025X050" value="100nF" x="41.9227" y="33.02" smashed="yes">
 <attribute name="NAME" x="44.7167" y="32.004" size="1.27" layer="25" ratio="10"/>
 <attribute name="VALUE" x="39.6367" y="30.226" size="1.27" layer="27" ratio="10"/>
 </element>
-<element name="C6" library="resistor" package="C025-025X050" value="" x="41.9227" y="35.560003125" smashed="yes">
+<element name="C6" library="resistor" package="C025-025X050" value="100nF" x="41.9227" y="35.560003125" smashed="yes">
 <attribute name="NAME" x="44.7167" y="35.814003125" size="1.27" layer="25" ratio="10"/>
 <attribute name="VALUE" x="39.6367" y="32.766003125" size="1.27" layer="27" ratio="10"/>
@@
 <attribute name="VALUE" x="72.7583" y="16.3322" size="1.778" layer="27" rot="R180"/>
 </element>
-<element name="C5" library="resistor" package="C025-025X050" value="" x="27.9527" y="39.2684" smashed="yes" rot="R90">
+<element name="C5" library="resistor" package="C025-025X050" value="100nF" x="27.9527" y="39.2684" smashed="yes" rot="R90">
 <attribute name="NAME" x="27.7749" y="44.5008" size="1.27" layer="25" ratio="10" rot="R270"/>
 <attribute name="VALUE" x="30.7467" y="36.9824" size="1.27" layer="27" ratio="10" rot="R90"/>
@@
 <attribute name="VALUE" x="25.7175" y="61.595" size="1.27" layer="27" rot="R180"/>
 </element>
-<element name="C10" library="resistor" package="C025-025X050" value="" x="24.4475" y="54.61" smashed="yes" rot="R90">
+<element name="C10" library="resistor" package="C025-025X050" value="100nF" x="24.4475" y="54.61" smashed="yes" rot="R90">
 <attribute name="NAME" x="26.924" y="55.8165" size="1.27" layer="25" ratio="10"/>
 <attribute name="VALUE" x="27.2415" y="52.324" size="1.27" layer="27" ratio="10" rot="R90"/>
 </element>
-<element name="R1" library="resistor" package="0207/10" value="" x="16.8275" y="53.34" smashed="yes" rot="R180">
+<element name="R1" library="resistor" package="0207/10" value="10k" x="16.8275" y="53.34" smashed="yes" rot="R180">
 <attribute name="NAME" x="13.1445" y="54.864" size="1.27" layer="25" ratio="10"/>
 <attribute name="VALUE" x="19.0881" y="53.975" size="1.27" layer="27" ratio="10" rot="R180"/>
 </element>
-<element name="Q3" library="crystal" package="HC18U-V" value="" x="25.7175" y="30.48" smashed="yes" rot="R270">
+<element name="Q3" library="crystal" package="HC18U-V" value="8MHz" x="25.7175" y="30.48" smashed="yes" rot="R270">
 <attribute name="OC_FARNELL" value="unknown" x="25.7175" y="30.48" size="1.778" layer="27" rot="R270" display="off"/>
 <attribute name="MF" value="" x="25.7175" y="30.48" size="1.778" layer="27" rot="R270" display="off"/>
@@
 <attribute name="VALUE" x="21.0947" y="35.56" size="1.27" layer="27" ratio="10" rot="R270"/>
 </element>
-<element name="C7" library="resistor" package="C025-025X050" value="" x="19.3675" y="33.02" smashed="yes" rot="R180">
+<element name="C7" library="resistor" package="C025-025X050" value="22pF" x="19.3675" y="33.02" smashed="yes" rot="R180">
 <attribute name="NAME" x="17.7165" y="35.814" size="1.27" layer="25" ratio="10"/>
 <attribute name="VALUE" x="21.6535" y="35.814" size="1.27" layer="27" ratio="10" rot="R180"/>
 </element>
-<element name="C8" library="resistor" package="C025-025X050" value="" x="19.3675" y="27.94" smashed="yes" rot="R180">
+<element name="C8" library="resistor" package="C025-025X050" value="22pF" x="19.3675" y="27.94" smashed="yes" rot="R180">
 <attribute name="NAME" x="17.7165" y="24.384" size="1.27" layer="25" ratio="10"/>
 <attribute name="VALUE" x="21.6535" y="30.734" size="1.27" layer="27" ratio="10" rot="R180"/>
@@
 <attribute name="VALUE" x="51.435" y="36.83" size="1.27" layer="27" rot="R90"/>
 </element>
-<element name="C9" library="resistor" package="C025-025X050" value="" x="44.45" y="8.89" smashed="yes" rot="R270">
+<element name="C9" library="resistor" package="C025-025X050" value="100nF" x="44.45" y="8.89" smashed="yes" rot="R270">
 <attribute name="NAME" x="43.434" y="6.096" size="1.27" layer="25" ratio="10" rot="R270"/>
 <attribute name="VALUE" x="41.656" y="11.176" size="1.27" layer="27" ratio="10" rot="R270"/>
 </element>
-<element name="C11" library="resistor" package="C025-025X050" value="" x="19.05" y="5.08" smashed="yes" rot="R90">
+<element name="C11" library="resistor" package="C025-025X050" value="100nF" x="19.05" y="5.08" smashed="yes" rot="R90">
 <attribute name="NAME" x="20.066" y="9.906" size="1.27" layer="25" ratio="10" rot="R180"/>
 <attribute name="VALUE" x="21.844" y="2.794" size="1.27" layer="27" ratio="10" rot="R90"/>
 </element>
-<element name="C12" library="resistor" package="C025-025X050" value="" x="12.7" y="19.05"/>
+<element name="C12" library="resistor" package="C025-025X050" value="100nF" x="12.7" y="19.05"/>
 <element name="JP2" library="pinhead" package="2X03" value="" x="27.94" y="6.35" smashed="yes" rot="R270">
 <attribute name="NAME" x="26.67" y="10.795" size="1.27" layer="25" ratio="10"/>
