File: PCB-Layouts/MoleNet_v5.0/MoleNet_v5.0.sch (EAGLE design)
At the start: 47 parts, among them J3 693072010801, Q1 MOSFET-NCHANNELBSS138, U1 STM32L073RZT6, U2 SN74LVC1G240DBVR, U3 MCP1703-1802E/DB, X1 8MHz, X2 32kHz, X3 R141426

Commit message: Schematic and PCB updated
Parts:
- added LED1, LED2: (no value), adafruit:LEDCHIPLED_0805
- added R5, R8: 220, resistor:R-EU_R0805
Connections:
- removed net PB5: JP3.1, U1.PB5
- new net LED2: LED2.A, U1.PB5
- new net N$7: LED1.C, R5.2
- new net N$8: LED2.C, R8.2
- net 3.3V: now also JP3.1, LED1.A
- net GND: now also R5.1, R8.1
Other:
- note added: "Debug LED"
- note added: "Last Updated: 23.03.2022"
- note removed: "Last Updated: 21.02.2022"
Changed lines of the file:
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@@
 <part name="U$31" library="Airquality_Sensor" library_urn="urn:adsk.eagle:library:16015176" deviceset="GND" device=""/>
 <part name="SUPPLY17" library="SparkFun-PowerSymbols" library_urn="urn:adsk.eagle:library:530" deviceset="3.3V" device=""/>
+<part name="LED1" library="adafruit" library_urn="urn:adsk.eagle:library:420" deviceset="LED" device="CHIPLED_0805" package3d_urn="urn:adsk.eagle:package:6240559/1"/>
+<part name="LED2" library="adafruit" library_urn="urn:adsk.eagle:library:420" deviceset="LED" device="CHIPLED_0805" package3d_urn="urn:adsk.eagle:package:6240559/1"/>
+<part name="SUPPLY18" library="SparkFun-PowerSymbols" library_urn="urn:adsk.eagle:library:530" deviceset="3.3V" device=""/>
+<part name="R5" library="resistor" library_urn="urn:adsk.eagle:library:348" deviceset="R-EU_" device="R0805" package3d_urn="urn:adsk.eagle:package:23553/2" value="220"/>
+<part name="U$32" library="Airquality_Sensor" library_urn="urn:adsk.eagle:library:16015176" deviceset="GND" device=""/>
+<part name="R8" library="resistor" library_urn="urn:adsk.eagle:library:348" deviceset="R-EU_" device="R0805" package3d_urn="urn:adsk.eagle:package:23553/2" value="220"/>
+<part name="U$33" library="Airquality_Sensor" library_urn="urn:adsk.eagle:library:16015176" deviceset="GND" device=""/>
+<part name="SUPPLY19" library="SparkFun-PowerSymbols" library_urn="urn:adsk.eagle:library:530" deviceset="3.3V" device=""/>
 </parts>
 <sheets>
 <sheet>
 <plain>
-<text x="182.88" y="7.62" size="1.778" layer="94">Last Updated: 21.02.2022</text>
+<text x="182.88" y="7.62" size="1.778" layer="94">Last Updated: 23.03.2022</text>
 <wire x1="96.64" y1="0" x2="97.32" y2="0" width="0.1524" layer="94"/>
 <text x="143.51" y="25.4" size="1.4224" layer="94">RFM ON/OFF</text>
@@
 <wire x1="125.73" y1="29.21" x2="125.73" y2="63.5" width="0.1524" layer="94" style="longdash"/>
 <text x="129.54" y="132.08" size="1.778" layer="94">Unused Pins</text>
+<text x="100.33" y="60.96" size="1.778" layer="94">Debug LED</text>
 </plain>
 <instances>
@@
 <instance part="SUPPLY17" gate="G$1" x="171.45" y="110.49" smashed="yes">
 <attribute name="VALUE" x="171.45" y="113.284" size="1.778" layer="96" align="bottom-center"/>
+</instance>
+<instance part="LED1" gate="G$1" x="114.3" y="53.34" smashed="yes">
+<attribute name="NAME" x="117.856" y="48.768" size="1.778" layer="95" rot="R90"/>
+<attribute name="VALUE" x="120.015" y="48.768" size="1.778" layer="96" rot="R90"/>
+</instance>
+<instance part="LED2" gate="G$1" x="99.06" y="53.34" smashed="yes">
+<attribute name="NAME" x="102.616" y="48.768" size="1.778" layer="95" rot="R90"/>
+<attribute name="VALUE" x="104.775" y="48.768" size="1.778" layer="96" rot="R90"/>
+</instance>
+<instance part="SUPPLY18" gate="G$1" x="116.84" y="55.88" smashed="yes">
+<attribute name="VALUE" x="111.76" y="56.134" size="1.778" layer="96" align="bottom-center"/>
+</instance>
+<instance part="R5" gate="G$1" x="114.3" y="41.91" smashed="yes" rot="R90">
+<attribute name="NAME" x="112.8014" y="40.64" size="1.778" layer="95" rot="R90"/>
+<attribute name="VALUE" x="117.602" y="40.64" size="1.778" layer="96" rot="R90"/>
+</instance>
+<instance part="U$32" gate="G$1" x="114.3" y="33.02" smashed="yes">
+<attribute name="VALUE" x="116.586" y="33.02" size="1.27" layer="96"/>
+</instance>
+<instance part="R8" gate="G$1" x="99.06" y="41.91" smashed="yes" rot="R90">
+<attribute name="NAME" x="97.5614" y="40.64" size="1.778" layer="95" rot="R90"/>
+<attribute name="VALUE" x="102.362" y="40.64" size="1.778" layer="96" rot="R90"/>
+</instance>
+<instance part="U$33" gate="G$1" x="99.06" y="33.02" smashed="yes">
+<attribute name="VALUE" x="101.346" y="33.02" size="1.27" layer="96"/>
+</instance>
+<instance part="SUPPLY19" gate="G$1" x="90.17" y="91.44" smashed="yes">
+<attribute name="VALUE" x="90.17" y="94.234" size="1.778" layer="96" align="bottom-center"/>
 </instance>
 </instances>
@@
 <junction x="142.24" y="102.87"/>
 </segment>
+<segment>
+<pinref part="R5" gate="G$1" pin="1"/>
+<pinref part="U$32" gate="G$1" pin="GND"/>
+<wire x1="114.3" y1="36.83" x2="114.3" y2="35.56" width="0.1524" layer="91"/>
+</segment>
+<segment>
+<pinref part="R8" gate="G$1" pin="1"/>
+<pinref part="U$33" gate="G$1" pin="GND"/>
+<wire x1="99.06" y1="36.83" x2="99.06" y2="35.56" width="0.1524" layer="91"/>
+</segment>
 </net>
 <net name="SWDIO" class="0">
@@
 <junction x="166.37" y="110.49"/>
 </segment>
+<segment>
+<pinref part="JP3" gate="A" pin="1"/>
+<wire x1="99.06" y1="90.17" x2="95.25" y2="90.17" width="0.1524" layer="91"/>
+<pinref part="SUPPLY19" gate="G$1" pin="3.3V"/>
+<wire x1="95.25" y1="90.17" x2="93.98" y2="90.17" width="0.1524" layer="91"/>
+<wire x1="90.17" y1="91.44" x2="90.17" y2="90.17" width="0.1524" layer="91"/>
+<wire x1="90.17" y1="90.17" x2="93.98" y2="90.17" width="0.1524" layer="91"/>
+</segment>
+<segment>
+<pinref part="LED1" gate="G$1" pin="A"/>
+<pinref part="SUPPLY18" gate="G$1" pin="3.3V"/>
+<wire x1="114.3" y1="55.88" x2="116.84" y2="55.88" width="0.1524" layer="91"/>
+</segment>
 </net>
 <net name="VDDA" class="0">
@@
 </segment>
 </net>
-<net name="PB5" class="0">
-<segment>
-<pinref part="U1" gate="G$1" pin="PB5"/>
-<wire x1="17.78" y1="43.18" x2="16.51" y2="43.18" width="0.1524" layer="91"/>
-<label x="11.43" y="43.18" size="1.778" layer="95"/>
-</segment>
-<segment>
-<pinref part="JP3" gate="A" pin="1"/>
-<wire x1="99.06" y1="90.17" x2="93.98" y2="90.17" width="0.1524" layer="91"/>
-<label x="88.9" y="90.17" size="1.778" layer="95"/>
-</segment>
-</net>
 <net name="PB4" class="0">
 <segment>
@@
 </segment>
 </net>
+<net name="N$7" class="0">
+<segment>
+<pinref part="LED1" gate="G$1" pin="C"/>
+<pinref part="R5" gate="G$1" pin="2"/>
+<wire x1="114.3" y1="48.26" x2="114.3" y2="46.99" width="0.1524" layer="91"/>
+</segment>
+</net>
+<net name="N$8" class="0">
+<segment>
+<pinref part="LED2" gate="G$1" pin="C"/>
+<pinref part="R8" gate="G$1" pin="2"/>
+<wire x1="99.06" y1="48.26" x2="99.06" y2="46.99" width="0.1524" layer="91"/>
+</segment>
+</net>
+<net name="LED2" class="0">
+<segment>
+<pinref part="U1" gate="G$1" pin="PB5"/>
+<wire x1="17.78" y1="43.18" x2="16.51" y2="43.18" width="0.1524" layer="91"/>
+<label x="10.16" y="43.18" size="1.778" layer="95"/>
+</segment>
+<segment>
+<pinref part="LED2" gate="G$1" pin="A"/>
+<wire x1="99.06" y1="55.88" x2="99.06" y2="58.42" width="0.1524" layer="91"/>
+<label x="91.44" y="57.15" size="1.778" layer="95"/>
+</segment>
+</net>
