File: PCB-Layouts/MoleNet_v5.0/MoleNet_v5.0.brd (EAGLE design)
At the start: 100 x 80 mm, 45 parts, among them Q1 MOSFET-NCHANNELBSS138, U1 STM32L073RZT6, U2 SN74LVC1G240DBVR, U3 MCP1703-1802E/DB, X1 8MHz, X2 32kHz, X3 R141426

Commit message: SD card added, unused pins organiged
Parts:
- added J3: 693072010801, Wurth_Connectors_WR-CRD:693072010801
- added J4: (no value), SparkFun-Connectors:1X05
- added JP5: PINHD-2X4, Connector:2X04
- added JP6, JP7: PINHD-2X10, Connector:2X10
- C11: value (none) -> 1uF
- JP1: value PINHD-2X3 -> PINHD-2X6; device Connector:2X03 -> Connector:2X06
- JP2: value (none) -> PINHD-2X3; device adafruit:1X03 -> Connector:2X03
- JP3: value PINHD-1X4 -> PINHD-2X8; device Connector:1X04 -> Connector:2X08
- moved JP1 391.6 mm to (-232.4, -539.8)
- moved JP3 130.2 mm to (-240.0, -549.9)
- moved JP2 40.7 mm to (-246.4, -539.8)
Connections:
- net RX/TX renamed RFM_RX/TX
- removed net NSS: U$18.5
- removed net SPI1_MISO: JP1.1, U1.22
- removed net SPI1_MISO_ON: JP1.2, U$18.2
- removed net SPI1_MOSI: JP1.3, U1.23
- removed net SPI1_MOSI_ON: JP1.4, U$18.3
- removed net SPI1_SCK: JP1.5, U1.21
- removed net SPI1_SCK_ON: JP1.6, U$18.4
- removed net USART2_CK: U1.20
- removed net USART2_RX: U1.17
- removed net USART2_TX: U1.16
- new net N$19: U1.54
- new net PA0: JP1.1, U1.14
- new net PA1: JP1.3, U1.15
- new net PA11: JP6.7, U1.44
- new net PA12: JP6.9, U1.45
- new net PA15: JP6.11, U1.50
- new net PA2: JP6.3, U1.16
- new net PA3: JP6.5, U1.17
- new net PA4: JP1.5, U1.20
- new net PB0: JP1.7, U1.26
- new net PB1: JP6.13, U1.27
- new net PB11: JP3.7, U1.30
- new net PB12: JP3.9, U1.33
- new net PB13: JP3.11, U1.34
- new net PB14: JP3.13, U1.35
- new net PB15: JP3.15, U1.36
- new net PB2: JP6.15, U1.28
- new net PB3: JP6.17, U1.55
- new net PB4: JP6.19, U1.56
- new net PB5: JP3.1, U1.57
- new net PB8: JP3.3, U1.61
- new net PB9: JP3.5, U1.62
- new net PC0: JP1.9, U1.8
- new net PC1: JP1.11, U1.9
- new net PC10: JP7.11, U1.51
- new net PC11: JP7.13, U1.52
- new net PC12: JP7.15, U1.53
- new net PC13: JP7.17, U1.2
- new net PC6: JP7.3, U1.37
- new net PC7: JP7.5, U1.38
- new net PC8: JP7.7, U1.39
- new net PC9: JP7.9, U1.40
- new net PD2: JP7.19
- new net RFM_CS: JP5.7, U1.25
- new net RFM_CS/ON: JP5.8, U$18.5
- new net RFM_MISO: JP5.1, U1.22
- new net RFM_MISO/ON: JP5.2, U$18.2
- new net RFM_MOSI: JP5.3, U1.23
- new net RFM_MOSI/ON: JP5.4, U$18.3
- new net RFM_SCK: JP5.5, U1.21
- new net RFM_SCK/ON: JP5.6, U$18.4
- new net SD_CS: J3.2, U1.24
- new net SD_MISO: J3.7, U1.10
- new net SD_MOSI: J3.3, U1.11
- new net SD_SCK: J3.5, U1.29
- net 3.3V: now also J3.4, J4.3, J4.4, JP2.1, JP6.1, JP7.1; no longer JP3.1
- net GND: now also J3.6, J4.1, J4.2, JP1.10, JP1.12, JP1.2, JP1.4, JP1.6, JP1.8, JP2.2, JP2.4, JP2.6, JP3.10, JP3.12, JP3.14, JP3.16, JP3.2, JP3.6, JP3.8, JP6.10, JP6.12, JP6.14, JP6.16, JP6.18, JP6.2, JP6.20, JP6.4, JP6.6, JP6.8, JP7.10, JP7.12, JP7.14, JP7.16, JP7.18, JP7.2, JP7.20, JP7.4, JP7.6, JP7.8
- net I2C1_SCL: now also JP2.3, U1.58; no longer JP3.2
- net I2C1_SDA: now also JP2.5, U1.59; no longer JP3.3
- net NRST: now also U$18.6
- net VIN: now also J4.5

Commit message: Schematic and PCB updated
Parts:
- removed U$1: (no value), SOT95P237X111-3N:SOT95P237X111-3N
- removed U$15: MCP1703_SOT23_3L, MCP1703_SOT23_3L:MCP1703_SOT23_3L
- removed U$4: STM32L053R8-LQFP64, STM32L053R8_LQFP64 (1):STM32L053R8-LQFP64
- added LED1, LED2: (no value), adafruit:CHIPLED_0805
- added R5, R8: 220, resistor:R0805
- moved J4 735.0 mm to (86.4, 76.2), turned to 180 degrees
- moved JP7 716.3 mm to (94.0, 64.8), turned to 90 degrees
- moved JP1 668.1 mm to (94.0, 43.2), turned to 90 degrees
- moved JP2 663.0 mm to (94.0, 29.2), turned to 90 degrees
- moved JP3 650.7 mm to (3.81, 53.3), turned to 90 degrees
- moved JP6 636.8 mm to (3.81, 29.2), turned to 90 degrees
- moved J3 602.1 mm to (40.6, 8.89)
- moved JP5 598.8 mm to (59.7, 15.2), turned to 270 degrees
- moved R4 570.3 mm to (35.6, 22.9), turned to 180 degrees
- moved J1 567.0 mm to (6.35, 72.4)
- moved C12 565.1 mm to (29.2, 5.08)
- moved D1 564.6 mm to (27.9, 14.0), turned to 90 degrees
- moved C18 558.3 mm to (91.4, 16.5), turned to 180 degrees
- moved R3 548.7 mm to (15.2, 15.2)
- moved R7 540.8 mm to (10.2, 15.2)
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Connections:
- removed net PB5: JP3.1, U1.57
- new net LED2: LED2.A, U1.57
- new net N$7: LED1.C, R5.2
- new net N$8: LED2.C, R8.2
- net 3.3V: now also JP3.1, LED1.A
- net GND: now also R5.1, R8.1
Other:
- board text added: "LED"
- board text added: "Power"
